File: femtosat/eagle.brd (EAGLE design)
At the start: 24.1 x 61 mm, 23 parts, among them U1 ATMEGA328P_TQFP, U2 915MHz, U3 3.3V/150mA, U4 9DoF IMU, U5 BME280, Y1 16MHz

Commit message: Changed Shaped
May need to shrink its width
Other:
- board size 24.1 x 61 mm -> 24.1 x 58.4 mm
Changed lines of the file:
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@@
 <board>
 <plain>
-<wire x1="17.408025" y1="70.221975" x2="21.961971875" y2="64.398028125" width="0.1524" layer="20"/>
-<wire x1="21.961971875" y1="64.398028125" x2="22.86" y2="59.163946875" width="0.1524" layer="20"/>
-<wire x1="22.86" y1="59.163946875" x2="22.86" y2="19.57605" width="0.1524" layer="20"/>
-<wire x1="22.86" y1="19.57605" x2="20.691975" y2="14.341975" width="0.1524" layer="20"/>
-<wire x1="20.691975" y1="14.341975" x2="19.948028125" y2="13.598028125" width="0.1524" layer="20"/>
-<wire x1="19.948028125" y1="13.598028125" x2="14.713946875" y2="11.43" width="0.1524" layer="20"/>
-<wire x1="14.713946875" y1="11.43" x2="6.87605" y2="11.43" width="0.1524" layer="20"/>
-<wire x1="6.87605" y1="11.43" x2="1.641975" y2="13.598025" width="0.1524" layer="20"/>
-<wire x1="1.641975" y1="13.598025" x2="0.898028125" y2="14.341971875" width="0.1524" layer="20"/>
-<wire x1="0.898028125" y1="14.341971875" x2="-1.27" y2="19.576053125" width="0.1524" layer="20"/>
-<wire x1="-1.27" y1="19.576053125" x2="-1.27" y2="59.16395" width="0.1524" layer="20"/>
-<wire x1="-1.27" y1="59.16395" x2="-0.371975" y2="64.398025" width="0.1524" layer="20"/>
-<wire x1="-0.371975" y1="64.398025" x2="4.181975" y2="70.221975" width="0.1524" layer="20"/>
-<wire x1="4.181975" y1="70.221975" x2="8.89" y2="72.39" width="0.1524" layer="20"/>
-<wire x1="8.89" y1="72.39" x2="12.7" y2="72.39" width="0.1524" layer="20"/>
-<wire x1="12.7" y1="72.39" x2="17.408025" y2="70.221975" width="0.1524" layer="20"/>
+<wire x1="22.86" y1="59.163946875" x2="22.86" y2="58.42" width="0.1524" layer="20"/>
+<wire x1="22.86" y1="58.42" x2="22.86" y2="15.24" width="0.1524" layer="20"/>
+<wire x1="-1.27" y1="64.77" x2="-1.27" y2="15.24" width="0.1524" layer="20"/>
+<wire x1="-1.27" y1="15.24" x2="2.54" y2="11.43" width="0.1524" layer="20"/>
+<wire x1="2.54" y1="11.43" x2="19.05" y2="11.43" width="0.1524" layer="20"/>
+<wire x1="19.05" y1="11.43" x2="22.86" y2="15.24" width="0.1524" layer="20"/>
 <text x="5.842" y="64.897" size="1.778" layer="1" font="vector">Angstrom</text>
 <text x="19.431" y="51.562" size="1.016" layer="1" font="vector">SCL</text>
 <text x="19.304" y="49.149" size="1.016" layer="1" font="vector">SDA</text>
+<wire x1="-1.27" y1="64.77" x2="3.81" y2="69.85" width="0.1524" layer="20"/>
+<wire x1="3.81" y1="69.85" x2="17.78" y2="69.85" width="0.1524" layer="20"/>
+<wire x1="17.78" y1="69.85" x2="22.86" y2="64.77" width="0.1524" layer="20"/>
+<wire x1="22.86" y1="64.77" x2="22.86" y2="59.163946875" width="0.1524" layer="20"/>
 </plain>
 <attributes>
